File: TechDevPCB/TechDevPCB.kicad_pcb (KiCad board)
At the start: 2 copper layers, 51 parts, among them J1 Screw_Terminal_01x02, J10 Conn_01x05_Pin, J11 Conn_01x01_Socket, J12 Screw_Terminal_01x04, J13 Conn_01x01_Socket, J14 Conn_01x01_Socket, J15 Conn_01x01_Socket, J16 Conn_01x01_Socket, J17 Conn_01x01_Socket, J18 Conn_01x01_Socket, J19 Conn_01x01_Socket, J2 Screw_Terminal_01x02, J20 Conn_01x01_Socket, J21 Conn_01x01_Socket, J22 Conn_01x01_Socket, J23 Conn_01x01_Socket, J24 Conn_01x01_Socket, J25 Conn_01x01_Socket, J26 Conn_01x01_Socket, J27 Conn_01x01_Socket, J28 Conn_01x01_Socket, J29 Conn_01x01_Socket, J3 Conn_01x02_Pin, J30 Conn_01x01_Socket, J31 Conn_01x01_Socket, J4 Screw_Terminal_01x04, J5 Conn_01x02_Pin, J6 Conn_01x05_Pin, J7 Conn_01x04_Pin, J8 Conn_01x05_Pin, J9 Conn_01x05_Pin, U1 DRV8825_STEPPER_MOTOR_DRIVER_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, U2 DRV8825_STEPPER_MOTOR_DRIVER_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, U3 XL6009 Boost Converter

Commit message: Created board
Parts:
- moved H2 72.7 mm to (150.2, 29.2)
- moved H1 71.5 mm to (150.2, 123.0)
- moved J8 70.2 mm to (144.7, 64.9)
- moved H4 69.2 mm to (79.5, 123.1)
- moved H3 67.8 mm to (79.5, 29.2)
- moved J4 33.1 mm to (83.3, 57.1)
- moved J3 27.7 mm to (97.4, 73.0), turned to -90 degrees
- moved J2 27.7 mm to (138.9, 30.5)
- moved J1 27.1 mm to (126.0, 30.5)
- moved C1 24.0 mm to (121.4, 70.6), turned to -90 degrees
- moved J12 21.5 mm to (83.3, 35.8)
- moved C2 18.9 mm to (115.6, 96.8)
- moved J9 18.2 mm to (144.7, 79.4)
- moved J5 16.5 mm to (97.5, 101.6), turned to -90 degrees
- moved J10 14.5 mm to (144.7, 104.0)
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Routing:
- net A0: track 0.00 -> 126.8 mm, vias 0 -> 1
- net A1: track 0.00 -> 120.3 mm, vias 0 -> 1
- net A2: track 0.00 -> 114.0 mm, vias 0 -> 1
- net +5V: track 0.00 -> 107.2 mm, vias 0 -> 1
- net D3: track 0.00 -> 103.8 mm, vias 0 -> 1
- net D2: track 0.00 -> 100.1 mm, vias 0 -> 1
- net +BATT: track 83.0 -> 165.6 mm
- net GND2: track 39.6 -> 111.1 mm
- net D9: track 0.00 -> 68.7 mm
- net D5: track 0.00 -> 66.9 mm
- net D10: track 0.00 -> 65.9 mm
- net D4: track 0.00 -> 64.8 mm
- net D11: track 0.00 -> 61.8 mm
- net +3.3V: track 0.00 -> 58.8 mm
- net D12: track 0.00 -> 57.7 mm
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Other:
- board outline added: 80.8 x 104.3 mm
- board text added: "A0"
- board text added: "A1"
- board text added: "A2"
- board text added: "AX 1 (24V)"
- board text added: "AX2 (BATT)"
- board text added: "AXIS 1 ^"
- board text added: "AXIS 2 ^"
- board text added: "B1"
- board text added: "B2"
- board text added: "D0"
- board text added: "D1"
- board text added: "D2"
- board text added: "D3"
- board text added: "D4"
- board text added: "D5"
- board text added: "D6"
- board text added: "D7"
- board text added: "D8"
- board text added: "EN"
- board text added: "FLT"
- board text added: "GND2"
- board text added: "Switch"

Commit message: PCB Updates
Routing:
- net GND2: track 111.1 -> 138.5 mm
- net GND: track 45.5 -> 62.9 mm
- net +BATT: track 165.6 -> 162.6 mm
- net +24V: track 56.1 -> 53.5 mm
- net D4: track 64.8 -> 63.7 mm

Commit message: PCB Updates
Parts:
- moved J12 23.4 mm to (83.3, 59.2)
- moved J4 21.3 mm to (83.3, 35.8)
- moved J2 0.25 mm to (138.7, 30.5)
Connections:
- J12 pad 1: AX1_B2 -> AX2_B2
- J12 pad 2: AX1_B1 -> AX2_B1
- J12 pad 3: AX1_A1 -> AX2_A1
- J12 pad 4: AX1_A2 -> AX2_A2
- J4 pad 1: AX2_B2 -> AX1_B2
- J4 pad 2: AX2_B1 -> AX1_B1
- J4 pad 3: AX2_A1 -> AX1_A1
- J4 pad 4: AX2_A2 -> AX1_A2
Routing:
- net +BATT: track 162.6 -> 159.8 mm
- net AX1_A1: track 64.1 -> 61.4 mm
- net AX1_A2: track 61.0 -> 58.7 mm
- net GND2: track 138.5 -> 140.4 mm
- net AX1_FLT: track 36.2 -> 34.3 mm
- net AX1_B1: track 65.8 -> 64.3 mm
- net AX1_B2: track 68.3 -> 67.3 mm
- net AX2_B2: track 75.2 -> 74.3 mm
- net AX2_B1: track 72.2 -> 71.4 mm
- net AX2_A2: track 66.8 -> 66.0 mm
- net AX2_A1: track 69.4 -> 68.5 mm
- net Net-(J1-Pin_2): track 20.2 -> 21.0 mm
Other:
- board text added: "+"
- board text added: "-"

Commit message: PCB Updates
Parts:
- removed H4: MountingHole, MountingHole:MountingHole_3.2mm_M3_DIN965
- added D1: LED, LED_THT:LED_Rectangular_W3.0mm_H2.0mm, F.Cu at (174.0, 138.0)
- added D2: LED, LED_THT:LED_Rectangular_W3.0mm_H2.0mm, F.Cu at (169.4, 138.2)
- added G***: LOGO, Footprints:QRET, F.Cu at (125.4, 50.8)
- added Q1: PMOS, Package_TO_SOT_THT:TO-251-3-1EP_Horizontal_TabDown, F.Cu at (141.0, 52.1)
- added R1: 30k, Resistor_THT:R_Axial_DIN0207_L6.3mm_D2.5mm_P10.16mm_Horizontal, F.Cu at (172.9, 65.1)
- added R2: 10k, Resistor_THT:R_Axial_DIN0207_L6.3mm_D2.5mm_P10.16mm_Horizontal, F.Cu at (167.6, 65.0)
- added R3: 500, Resistor_THT:R_Axial_DIN0207_L6.3mm_D2.5mm_P10.16mm_Horizontal, F.Cu at (181.0, 123.9)
- added R4: 500, Resistor_THT:R_Axial_DIN0207_L6.3mm_D2.5mm_P10.16mm_Horizontal, F.Cu at (185.7, 123.8)
- moved J4 68.8 mm to (113.6, 97.6)
- moved J12 68.6 mm to (113.6, 120.7)
- moved H1 38.1 mm to (184.4, 139.7)
- moved C2 37.1 mm to (149.8, 111.0)
- moved J9 37.1 mm to (178.9, 93.6)
- moved J10 37.1 mm to (178.9, 118.2)
- moved J29 37.1 mm to (133.8, 134.4)
- moved J6 37.1 mm to (178.9, 63.5)
- moved J7 37.1 mm to (178.9, 59.7)
- moved J8 37.1 mm to (178.9, 79.1)
- moved JP9 37.1 mm to (130.2, 134.4)
- moved J1 37.1 mm to (160.2, 44.7)
- moved J13 37.1 mm to (133.8, 91.2)
- moved J15 37.1 mm to (133.8, 94.9)
- moved J17 37.1 mm to (133.8, 98.6)
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Connections:
- J1 pad 1: +BATT -> Net-(J1-Pin_1)
Routing:
- net A7: track 9.05 -> 66.4 mm
- net GND: track 62.9 -> 103.8 mm, vias 0 -> 4
- net Net-(J1-Pin_1): track 0.00 -> 23.6 mm
- net Net-(D2-A): track 0.00 -> 21.8 mm
- net GND2: track 140.4 -> 159.7 mm, vias 0 -> 4
- net AX2_A2: track 66.0 -> 50.9 mm
- net AX2_A1: track 68.5 -> 54.2 mm
- net AX1_B2: track 67.3 -> 53.6 mm
- net AX1_A1: track 61.4 -> 48.6 mm
- net AX1_A2: track 58.7 -> 46.3 mm
- net AX2_B2: track 74.3 -> 63.0 mm
- net AX2_B1: track 71.4 -> 60.4 mm
- net D12: track 57.7 -> 67.7 mm
- net AX1_B1: track 64.3 -> 55.7 mm
- net AX2_FLT: track 35.0 -> 42.0 mm
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Other:
- board size 80.8 x 104.3 mm -> 85.4 x 106.8 mm
- board text added: "10k"
- board text added: "500"
- board text added: "BATTERY STATUS"
- board text added: "Tech Dev '23/24"
- board text removed: "AXIS 1 ^"

Commit message: PCB Updates
Routing:
- net D2: track 101.1 -> 100.1 mm, vias 2 -> 1
- net D3: track 104.6 -> 103.8 mm, vias 2 -> 1
Changed lines of the file:
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@@
     (effects (font (size 1.5 1.5) (thickness 0.3) bold) (justify left bottom))
+  )
+  (gr_text "-" (at 173.5582 140.1064) (layer "F.SilkS")
+    (effects (font (size 1 1) (thickness 0.15)))
   )
   (gr_text "B1" (at 119.1514 126.8984) (layer "F.SilkS")
@@
     (effects (font (size 1.5 1.5) (thickness 0.3) bold) (justify left bottom))
   )
+  (gr_text "+" (at 166.624 140.081) (layer "F.SilkS")
+    (effects (font (size 1 1) (thickness 0.15)))
+  )
   (gr_text "A1" (at 119.1514 131.9784) (layer "F.SilkS")
     (effects (font (size 1.5 1.5) (thickness 0.3) bold) (justify left bottom))
@@
     (effects (font (size 1.5 1.5) (thickness 0.3) bold) (justify left bottom))
   )
+  (gr_text "+" (at 176.6316 140.0302) (layer "F.SilkS")
+    (effects (font (size 1 1) (thickness 0.15)))
+  )
   (gr_text "D4" (at 122.2756 135.3566) (layer "F.SilkS")
     (effects (font (size 1.5 1.5) (thickness 0.3) bold) (justify left bottom))
@@
   (gr_text "+24V" (at 180.5178 55.499) (layer "F.SilkS")
     (effects (font (size 1.5 1.5) (thickness 0.3) bold) (justify left bottom))
+  )
+  (gr_text "-" (at 169.5958 140.1064) (layer "F.SilkS")
+    (effects (font (size 1 1) (thickness 0.15)))
   )
   (gr_text "D11" (at 180.7718 99.695) (layer "F.SilkS")
@@
   (segment (start 149.1996 107.7722) (end 150.7998 106.172) (width 0.5) (layer "B.Cu") (net 4))
   (segment (start 166.9542 129.5146) (end 166.9542 103.886) (width 0.5) (layer "B.Cu") (net 4))
-  (segment (start 124.435902 137.668) (end 152.8826 137.668) (width 0.3) (layer "F.Cu") (net 5))
   (segment (start 123.3678 109.22) (end 123.3678 136.599898) (width 0.3) (layer "F.Cu") (net 5))
+  (segment (start 124.435902 137.668) (end 151.883417 137.668) (width 0.3) (layer "F.Cu") (net 5))
   (segment (start 129.5608 105.918) (end 126.6698 105.918) (width 0.3) (layer "F.Cu") (net 5))
+  (segment (start 151.883417 137.668) (end 151.895917 137.6555) (width 0.3) (layer "F.Cu") (net 5))
+  (segment (start 123.3678 136.599898) (end 124.435902 137.668) (width 0.3) (layer "F.Cu") (net 5))
   (segment (start 126.6698 105.918) (end 123.3678 109.22) (width 0.3) (layer "F.Cu") (net 5))
-  (segment (start 123.3678 136.599898) (end 124.435902 137.668) (width 0.3) (layer "F.Cu") (net 5))
-  (via (at 152.654 137.668) (size 0.8) (drill 0.4) (layers "F.Cu" "B.Cu") (net 5))
-  (via (at 151.8666 137.6555) (size 0.8) (drill 0.4) (layers "F.Cu" "B.Cu") (net 5))
-  (segment (start 151.8666 137.6555) (end 153.0983 137.6555) (width 0.3) (layer "B.Cu") (net 5))
+  (via (at 151.895917 137.6555) (size 0.8) (drill 0.4) (layers "F.Cu" "B.Cu") (net 5))
+  (segment (start 153.0983 137.6555) (end 153.8478 136.906) (width 0.3) (layer "B.Cu") (net 5))
+  (segment (start 151.895917 137.6555) (end 153.0983 137.6555) (width 0.3) (layer "B.Cu") (net 5))
   (segment (start 153.8478 106.426) (end 156.2608 104.013) (width 0.3) (layer "B.Cu") (net 5))
-  (segment (start 153.0983 137.6555) (end 153.8478 136.906) (width 0.3) (layer "B.Cu") (net 5))
   (segment (start 153.8478 136.906) (end 153.8478 106.426) (width 0.3) (layer "B.Cu") (net 5))
+  (segment (start 122.6678 136.889848) (end 122.6678 106.237) (width 0.3) (layer "F.Cu") (net 6))
   (segment (start 156.2608 106.7549) (end 156.2608 106.553) (width 0.5) (layer "F.Cu") (net 6))
+  (segment (start 129.5608 102.235) (end 126.6698 102.235) (width 0.3) (layer "F.Cu") (net 6))
+  (segment (start 122.6678 106.237) (end 126.6698 102.235) (width 0.3) (layer "F.Cu") (net 6))
+  (segment (start 152.527 138.43) (end 124.207952 138.43) (width 0.3) (layer "F.Cu") (net 6))
   (segment (start 124.207952 138.43) (end 122.6678 136.889848) (width 0.3) (layer "F.Cu") (net 6))
-  (segment (start 122.6678 106.237) (end 126.6698 102.235) (width 0.3) (layer "F.Cu") (net 6))
-  (segment (start 153.321176 138.412232) (end 153.303408 138.43) (width 0.3) (layer "F.Cu") (net 6))
-  (segment (start 122.6678 136.889848) (end 122.6678 106.237) (width 0.3) (layer "F.Cu") (net 6))
-  (segment (start 129.5608 102.235) (end 126.6698 102.235) (width 0.3) (layer "F.Cu") (net 6))
-  (segment (start 153.303408 138.43) (end 124.207952 138.43) (width 0.3) (layer "F.Cu") (net 6))
   (via (at 152.527 138.43) (size 0.8) (drill 0.4) (layers "F.Cu" "B.Cu") (net 6))
-  (via (at 153.321176 138.412232) (size 0.8) (drill 0.4) (layers "F.Cu" "B.Cu") (net 6))
   (segment (start 154.3558 108.458) (end 156.2608 106.553) (width 0.3) (layer "B.Cu") (net 6))
+  (segment (start 154.3558 137.377608) (end 153.303408 138.43) (width 0.3) (layer "B.Cu") (net 6))
   (segment (start 154.3558 137.377608) (end 154.3558 108.458) (width 0.3) (layer "B.Cu") (net 6))
   (segment (start 153.303408 138.43) (end 152.527 138.43) (width 0.3) (layer "B.Cu") (net 6))
-  (segment (start 153.321176 138.412232) (end 154.3558 137.377608) (width 0.3) (layer "B.Cu") (net 6))
-  (segment (start 153.321176 138.412232) (end 153.303408 138.43) (width 0.3) (layer "B.Cu") (net 6))
   (segment (start 129.5608 134.366) (end 126.6698 134.366) (width 0.3) (layer "F.Cu") (net 7))
   (segment (start 126.6698 134.366) (end 124.8918 134.366) (width 0.3) (layer "F.Cu") (net 7))

Commit message: Updates
Parts:
- removed G***: LOGO, Footprints:QRET
- added J32: Conn_01x04_Pin, Connector_PinHeader_2.54mm:PinHeader_1x04_P2.54mm_Vertical, F.Cu at (153.8, 141.7)
Routing:
- net GND2: track 159.7 -> 187.5 mm, vias 4 -> 8
- net GND: track 103.8 -> 120.7 mm, vias 4 -> 8
- net D4: track 63.0 -> 59.4 mm
- net AX2_B1: track 60.4 -> 58.9 mm
- net D5: track 66.3 -> 65.1 mm
- net AX1_B2: track 53.6 -> 54.6 mm
- net A1: track 120.3 -> 121.1 mm
- net A2: track 114.0 -> 114.7 mm
- net +5V: track 107.3 -> 106.6 mm
- net D10: track 65.9 -> 65.2 mm
- net A0: track 126.8 -> 127.5 mm
Other:
- outline, holes or cut-outs redrawn
- board text added: "GND"
- board text added: "STS Control Board March 21 2024 (Rev 1.0)"
- board text added: "Teighin Nordholt"
