File: TechDevPCB/TechDevPCB.kicad_sch (KiCad schematic)
At the start: 15 parts, among them J1 Screw_Terminal_01x02, J10 Conn_01x05_Pin, J2 Screw_Terminal_01x02, J3 Conn_01x02_Pin, J4 Conn_01x04_Pin, J5 Conn_01x02_Pin, J6 Conn_01x04_Pin, J8 Conn_01x05_Pin, J9 Conn_01x05_Pin, U1 DRV8825_STEPPER_MOTOR_DRIVER_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, U2 DRV8825_STEPPER_MOTOR_DRIVER_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, U3 XL6009 Boost Converter

Commit message: PCB Updates
Parts:
- removed J4, J6: Conn_01x04_Pin, Connector_PinHeader_2.54mm:PinHeader_1x04_P2.54mm_Vertical, symbol Connector:Conn_01x04_Pin
- added H1, H2, H3, H4: MountingHole, MountingHole:MountingHole_3.2mm_M3_DIN965, symbol Mechanical:MountingHole
- added J11, J13, J14, J15, J16, J17, J18, J19, J20, J21, J22, J23, J24, J25, J26, J27, J28, J29, J30, J31: Conn_01x01_Socket, Connector_PinHeader_2.54mm:PinHeader_1x01_P2.54mm_Vertical, symbol Connector:Conn_01x01_Socket
- added J12, J4: Screw_Terminal_01x04, TerminalBlock:TerminalBlock_bornier-4_P5.08mm, symbol Connector:Screw_Terminal_01x04
- added J6: Conn_01x05_Pin, Connector_PinHeader_2.54mm:PinHeader_1x05_P2.54mm_Vertical, symbol Connector:Conn_01x05_Pin
- added J7: Conn_01x04_Pin, Connector_PinHeader_2.54mm:PinHeader_1x04_P2.54mm_Vertical, symbol Connector:Conn_01x04_Pin
- added JP1, JP10, JP2, JP3, JP4, JP5, JP6, JP7, JP8, JP9: SolderJumper_2_Open, Jumper:SolderJumper-2_P1.3mm_Open_Pad1.0x1.5mm, symbol Jumper:SolderJumper_2_Open
- J2: footprint (none) -> TerminalBlock:TerminalBlock_bornier-2_P5.08mm
Connections:
- net +24V: now also J7.3 (Pin_3), J7.4 (Pin_4)
- net +3.3V: now also J6.4 (Pin_4), J6.5 (Pin_5)
- net +5V: now also J6.2 (Pin_2), J6.3 (Pin_3)
- net +BATT: now also J7.1 (Pin_1), J7.2 (Pin_2)
- net A0: now also J11.1 (Pin_1), J22.1 (Pin_1), JP1.1 (A), JP6.1 (A); no longer U1.2 (M0), U2.2 (M0)
- net A1: now also J14.1 (Pin_1), J26.1 (Pin_1), JP2.1 (A), JP8.1 (A); no longer U1.3 (M1), U2.3 (M1)
- net A2: now also J16.1 (Pin_1), J24.1 (Pin_1), JP3.1 (A), JP7.1 (A); no longer U1.4 (M2), U2.4 (M2)
- net AX1_A1: now also J12.3 (Pin_3)
- net AX1_A2: now also J12.4 (Pin_4)
- net AX1_B1: now also J12.2 (Pin_2)
- net AX1_B2: now also J12.1 (Pin_1)
- net AX2_A1: now also J4.3 (Pin_3)
- net AX2_A2: now also J4.4 (Pin_4)
- net AX2_B1: now also J4.2 (Pin_2)
- net AX2_B2: now also J4.1 (Pin_1)
- net D0: now also J8.2 (Pin_2); no longer J8.1 (Pin_1)
- net D1: now also J8.1 (Pin_1); no longer J8.2 (Pin_2)
- net D2: now also J20.1 (Pin_1), JP5.1 (A); no longer U1.8 (DIR)
- net D3: now also J18.1 (Pin_1), JP4.1 (A); no longer U1.7 (STEP)
- net D4: now also J28.1 (Pin_1), JP9.1 (A); no longer U2.8 (DIR)
- net D5: now also J30.1 (Pin_1), JP10.1 (A); no longer U2.7 (STEP)
- net VIN: now also J6.1 (Pin_1)
- new net AX1_DIR: J21.1 (Pin_1), JP5.2 (B), U1.8 (DIR)
- new net AX1_M0: J13.1 (Pin_1), JP1.2 (B), U1.2 (M0)
- new net AX1_M1: J15.1 (Pin_1), JP2.2 (B), U1.3 (M1)
- new net AX1_M2: J17.1 (Pin_1), JP3.2 (B), U1.4 (M2)
- new net AX1_STEP: J19.1 (Pin_1), JP4.2 (B), U1.7 (STEP)
- new net AX2_DIR: J29.1 (Pin_1), JP9.2 (B), U2.8 (DIR)
- new net AX2_M0: J23.1 (Pin_1), JP6.2 (B), U2.2 (M0)
- new net AX2_M1: J27.1 (Pin_1), JP8.2 (B), U2.3 (M1)
- new net AX2_M2: J25.1 (Pin_1), JP7.2 (B), U2.4 (M2)
- new net AX2_STEP: J31.1 (Pin_1), JP10.2 (B), U2.7 (STEP)
Other:
- note added: "Axis 1 Motor Driver Solder Bridges"
- note added: "Axis 2 Motor Driver Solder Bridges"
- note added: "M3 Mounting Holes"
- note added: "Q: Solder bridge for sleep, rst pins of motor drivers?"
- note added: "Voltage Outs"
- note removed: "-Screw terminals for motor coils -Pin out for all voltages"
- moved on the sheet: A1, C1, J2, J5, U1, U2, U3

Commit message: Created board
Other:
- note added: "INCREASE TRACE WIDTH FOR BATT IN"
- note removed: "Q: Solder bridge for sleep, rst pins of motor drivers?"
Changed lines of the file:
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@@
     (effects (font (size 1.27 1.27)) (justify left bottom))
   )
-  (text "Q: Solder bridge for sleep, rst pins of motor drivers?\n"
-    (at 181.61 160.02 0)
+  (text "INCREASE TRACE WIDTH FOR BATT IN" (at 181.61 160.02 0)
     (effects (font (size 1.27 1.27)) (justify left bottom))
   )

Commit message: PCB Updates
Other:
- note added: "Research trace width Revise naming using Carter convention Delete screw terminals from schematic and board, put back in"
- note removed: "INCREASE TRACE WIDTH FOR BATT IN"
Changed lines of the file:
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@@
     (effects (font (size 1.27 1.27)) (justify left bottom))
   )
-  (text "INCREASE TRACE WIDTH FOR BATT IN" (at 181.61 160.02 0)
+  (text "Research trace width\nRevise naming using Carter convention\nDelete screw terminals from schematic and board, put back in\n"
+    (at 181.61 163.83 0)
     (effects (font (size 1.27 1.27)) (justify left bottom))
   )

Commit message: PCB Updates
Connections:
- net AX1_A1: now also J4.3 (Pin_3); no longer J12.3 (Pin_3)
- net AX1_A2: now also J4.4 (Pin_4); no longer J12.4 (Pin_4)
- net AX1_B1: now also J4.2 (Pin_2); no longer J12.2 (Pin_2)
- net AX1_B2: now also J4.1 (Pin_1); no longer J12.1 (Pin_1)
- net AX2_A1: now also J12.3 (Pin_3); no longer J4.3 (Pin_3)
- net AX2_A2: now also J12.4 (Pin_4); no longer J4.4 (Pin_4)
- net AX2_B1: now also J12.2 (Pin_2); no longer J4.2 (Pin_2)
- net AX2_B2: now also J12.1 (Pin_1); no longer J4.1 (Pin_1)

Commit message: PCB Updates
Parts:
- removed H4: MountingHole, MountingHole:MountingHole_3.2mm_M3_DIN965, symbol Mechanical:MountingHole
- added D1, D2: LED, LED_THT:LED_Rectangular_W3.0mm_H2.0mm, symbol Device:LED
- added Q1: PMOS, Package_TO_SOT_THT:TO-251-3-1EP_Horizontal_TabDown, symbol Simulation_SPICE:PMOS
- added R1: 30k, Resistor_THT:R_Axial_DIN0207_L6.3mm_D2.5mm_P10.16mm_Horizontal, symbol Device:R
- added R2: 10k, Resistor_THT:R_Axial_DIN0207_L6.3mm_D2.5mm_P10.16mm_Horizontal, symbol Device:R
- added R3, R4: 500, Resistor_THT:R_Axial_DIN0207_L6.3mm_D2.5mm_P10.16mm_Horizontal, symbol Device:R
Connections:
- net +BATT: now also Q1.3 (S), R1.1; no longer J1.1 (Pin_1)
- net A7: now also R1.2, R2.1
- net D12: now also R4.1
- net D13: now also R3.1
- net GND: now also D1.1 (K), D2.1 (K)
- net GND2: now also Q1.2 (G), R2.2
- new net: D1.2 (A), R3.2
- new net: D2.2 (A), R4.2
- new net: J1.1 (Pin_1), Q1.1 (D)
Other:
- note added: "Battery Monitor"
- note removed: "Research trace width Revise naming using Carter convention Delete screw terminals from schematic and board, put back in"
- moved on the sheet: H1, H2, H3

Commit message: PCB Updates
Other:
- moved on the sheet: D1, D2, R3, R4
Changed lines of the file:
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@@
     (fill (type none))
   )
-  (rectangle (start 176.53 83.185) (end 207.264 124.333)
+  (rectangle (start 176.53 83.185) (end 234.315 124.333)
     (stroke (width 0) (type dash))
     (fill (type none))
@@
     )
   )
-  (global_label "D13" (shape input) (at 211.455 91.44 90) (fields_autoplaced)
-    (effects (font (size 1.27 1.27)) (justify left))
-    (property "Intersheetrefs" "${INTERSHEET_REFS}" (at 211.455 84.7658 90)
+  (global_label "D13" (shape input) (at 211.455 94.615 90) (fields_autoplaced)
+    (effects (font (size 1.27 1.27)) (justify left))
+    (property "Intersheetrefs" "${INTERSHEET_REFS}" (at 211.455 87.9408 90)
       (effects (font (size 1.27 1.27)) (justify left) hide)
     )
@@
     )
   )
-  (global_label "D12" (shape input) (at 223.52 91.44 90) (fields_autoplaced)
-    (effects (font (size 1.27 1.27)) (justify left))
-    (property "Intersheetrefs" "${INTERSHEET_REFS}" (at 223.52 84.7658 90)
+  (global_label "D12" (shape input) (at 223.52 94.615 90) (fields_autoplaced)
+    (effects (font (size 1.27 1.27)) (justify left))
+    (property "Intersheetrefs" "${INTERSHEET_REFS}" (at 223.52 87.9408 90)
       (effects (font (size 1.27 1.27)) (justify left) hide)
     )
@@
     )
   )
-  (symbol (lib_id "Device:R") (at 211.455 95.25 0) (unit 1)
-    (in_bom yes) (on_board yes) (dnp no) (fields_autoplaced)
-    (property "Reference" "R3" (at 213.36 93.98 0)
-      (effects (font (size 1.27 1.27)) (justify left))
-    )
-    (property "Value" "500" (at 213.36 96.52 0)
-      (effects (font (size 1.27 1.27)) (justify left))
-    )
-    (property "Footprint" "Resistor_THT:R_Axial_DIN0207_L6.3mm_D2.5mm_P10.16mm_Horizontal" (at 209.677 95.25 90)
-      (effects (font (size 1.27 1.27)) hide)
-    )
-    (property "Datasheet" "~" (at 211.455 95.25 0)
+  (symbol (lib_id "Device:R") (at 211.455 98.425 0) (unit 1)
+    (in_bom yes) (on_board yes) (dnp no) (fields_autoplaced)
+    (property "Reference" "R3" (at 213.36 97.155 0)
+      (effects (font (size 1.27 1.27)) (justify left))
+    )
+    (property "Value" "500" (at 213.36 99.695 0)
+      (effects (font (size 1.27 1.27)) (justify left))
+    )
+    (property "Footprint" "Resistor_THT:R_Axial_DIN0207_L6.3mm_D2.5mm_P10.16mm_Horizontal" (at 209.677 98.425 90)
+      (effects (font (size 1.27 1.27)) hide)
+    )
+    (property "Datasheet" "~" (at 211.455 98.425 0)
       (effects (font (size 1.27 1.27)) hide)
     )
@@
     )
   )
-  (symbol (lib_id "Device:R") (at 223.52 95.25 0) (unit 1)
-    (in_bom yes) (on_board yes) (dnp no) (fields_autoplaced)
-    (property "Reference" "R4" (at 225.425 93.98 0)
-      (effects (font (size 1.27 1.27)) (justify left))
-    )
-    (property "Value" "500" (at 225.425 96.52 0)
-      (effects (font (size 1.27 1.27)) (justify left))
-    )
-    (property "Footprint" "Resistor_THT:R_Axial_DIN0207_L6.3mm_D2.5mm_P10.16mm_Horizontal" (at 221.742 95.25 90)
-      (effects (font (size 1.27 1.27)) hide)
-    )
-    (property "Datasheet" "~" (at 223.52 95.25 0)
+  (symbol (lib_id "Device:R") (at 223.52 98.425 0) (unit 1)
+    (in_bom yes) (on_board yes) (dnp no) (fields_autoplaced)
+    (property "Reference" "R4" (at 225.425 97.155 0)
+      (effects (font (size 1.27 1.27)) (justify left))
+    )
+    (property "Value" "500" (at 225.425 99.695 0)
+      (effects (font (size 1.27 1.27)) (justify left))
+    )
+    (property "Footprint" "Resistor_THT:R_Axial_DIN0207_L6.3mm_D2.5mm_P10.16mm_Horizontal" (at 221.742 98.425 90)
+      (effects (font (size 1.27 1.27)) hide)
+    )
+    (property "Datasheet" "~" (at 223.52 98.425 0)
       (effects (font (size 1.27 1.27)) hide)
     )
@@
     )
   )
-  (symbol (lib_id "Device:LED") (at 223.52 102.87 90) (unit 1)
-    (in_bom yes) (on_board yes) (dnp no) (fields_autoplaced)
-    (property "Reference" "D2" (at 226.695 103.1875 90)
+  (symbol (lib_id "Device:LED") (at 223.52 106.045 90) (unit 1)
+    (in_bom yes) (on_board yes) (dnp no) (fields_autoplaced)
+    (property "Reference" "D2" (at 226.695 106.3625 90)
       (effects (font (size 1.27 1.27)) (justify right))
     )
-    (property "Value" "LED" (at 226.695 105.7275 90)
+    (property "Value" "LED" (at 226.695 108.9025 90)
       (effects (font (size 1.27 1.27)) (justify right))
     )
-    (property "Footprint" "LED_THT:LED_Rectangular_W3.0mm_H2.0mm" (at 223.52 102.87 0)
-      (effects (font (size 1.27 1.27)) hide)
-    )
-    (property "Datasheet" "~" (at 223.52 102.87 0)
+    (property "Footprint" "LED_THT:LED_Rectangular_W3.0mm_H2.0mm" (at 223.52 106.045 0)
+      (effects (font (size 1.27 1.27)) hide)
+    )
+    (property "Datasheet" "~" (at 223.52 106.045 0)
       (effects (font (size 1.27 1.27)) hide)
     )
@@
     )
   )
-  (symbol (lib_id "power:GND") (at 223.52 106.68 0) (unit 1)
-    (in_bom yes) (on_board yes) (dnp no) (fields_autoplaced)
-    (property "Reference" "#PWR033" (at 223.52 113.03 0)
-      (effects (font (size 1.27 1.27)) hide)
-    )
-    (property "Value" "GND" (at 223.52 111.76 0)
-      (effects (font (size 1.27 1.27)))
-    )
-    (property "Footprint" "" (at 223.52 106.68 0)
-      (effects (font (size 1.27 1.27)) hide)
-    )
-    (property "Datasheet" "" (at 223.52 106.68 0)
+  (symbol (lib_id "power:GND") (at 223.52 109.855 0) (unit 1)
+    (in_bom yes) (on_board yes) (dnp no) (fields_autoplaced)
+    (property "Reference" "#PWR033" (at 223.52 116.205 0)
+      (effects (font (size 1.27 1.27)) hide)
+    )
+    (property "Value" "GND" (at 223.52 114.935 0)
+      (effects (font (size 1.27 1.27)))
+    )
+    (property "Footprint" "" (at 223.52 109.855 0)
+      (effects (font (size 1.27 1.27)) hide)
+    )
+    (property "Datasheet" "" (at 223.52 109.855 0)
       (effects (font (size 1.27 1.27)) hide)
     )
@@
     )
   )
-  (symbol (lib_id "power:GND") (at 211.455 106.68 0) (unit 1)
-    (in_bom yes) (on_board yes) (dnp no) (fields_autoplaced)
-    (property "Reference" "#PWR032" (at 211.455 113.03 0)
-      (effects (font (size 1.27 1.27)) hide)
-    )
-    (property "Value" "GND" (at 211.455 111.76 0)
-      (effects (font (size 1.27 1.27)))
-    )
-    (property "Footprint" "" (at 211.455 106.68 0)
-      (effects (font (size 1.27 1.27)) hide)
-    )
-    (property "Datasheet" "" (at 211.455 106.68 0)
+  (symbol (lib_id "power:GND") (at 211.455 109.855 0) (unit 1)
+    (in_bom yes) (on_board yes) (dnp no) (fields_autoplaced)
+    (property "Reference" "#PWR032" (at 211.455 116.205 0)
+      (effects (font (size 1.27 1.27)) hide)
+    )
+    (property "Value" "GND" (at 211.455 114.935 0)
+      (effects (font (size 1.27 1.27)))
+    )
+    (property "Footprint" "" (at 211.455 109.855 0)
+      (effects (font (size 1.27 1.27)) hide)
+    )
+    (property "Datasheet" "" (at 211.455 109.855 0)
       (effects (font (size 1.27 1.27)) hide)
     )
@@
     )
   )
-  (symbol (lib_id "Device:LED") (at 211.455 102.87 90) (unit 1)
-    (in_bom yes) (on_board yes) (dnp no) (fields_autoplaced)
-    (property "Reference" "D1" (at 214.63 103.1875 90)
+  (symbol (lib_id "Device:LED") (at 211.455 106.045 90) (unit 1)
+    (in_bom yes) (on_board yes) (dnp no) (fields_autoplaced)
+    (property "Reference" "D1" (at 214.63 106.3625 90)
       (effects (font (size 1.27 1.27)) (justify right))
     )
-    (property "Value" "LED" (at 214.63 105.7275 90)
+    (property "Value" "LED" (at 214.63 108.9025 90)
       (effects (font (size 1.27 1.27)) (justify right))
     )
-    (property "Footprint" "LED_THT:LED_Rectangular_W3.0mm_H2.0mm" (at 211.455 102.87 0)
-      (effects (font (size 1.27 1.27)) hide)
-    )
-    (property "Datasheet" "~" (at 211.455 102.87 0)
-      (effects (font (size 1.27 1.27)) hide)
-    )
+    (property "Footprint" "LED_THT:LED_Rectangular_W3.0mm_H2.0mm" (at 211.455 106.045 0)
+      (effects (font (size 1.27 1.27)) hide)
+    )
+    (property "Datasheet" "~" (at 211.455 106.045 0)
+      (effects (font (size 1.27 1.27)) hide)
+    )

Commit message: Updates
Parts:
- added J32: Conn_01x04_Pin, Connector_PinHeader_2.54mm:PinHeader_1x04_P2.54mm_Vertical, symbol Connector:Conn_01x04_Pin
Connections:
- net GND: now also J32.1 (Pin_1), J32.2 (Pin_2)
- net GND2: now also J32.3 (Pin_3), J32.4 (Pin_4)
Other:
- moved on the sheet: C1, U1
